File: pe/riddhi-buck-converter/riddhi-buck-converter.kicad_sch (KiCad schematic)
At the start: 0 parts

Commit message: PE Activity 3: MP1477 buck schematic and PCB import.
Parts:
- added C2, C4: 22uF, Capacitor_SMD:C_0603_1608Metric, symbol Device:C
- added C3: 10uF, Capacitor_SMD:C_0603_1608Metric, symbol Device:C
- added C5: 100nF, Capacitor_SMD:C_0603_1608Metric, symbol Device:C
- added L1: 2.2uH, Inductor_SMD:L_Sunlord_SWPA4020S, symbol Device:L
- added R1: 52.3k, Resistor_SMD:R_0603_1608Metric, symbol Device:R
- added R2: 10k, Resistor_SMD:R_0603_1608Metric, symbol Device:R
- added U1: MP1477HGTF-Z, Package_TO_SOT_SMD:SOT-563, symbol MP1470
Connections:
- new net: C5.1, C5.2, L1.1, U1.2 (SW)
- new net +12V: C3.2, U1.3 (IN), U1.5 (EN)
- new net +5V: C2.2, C4.2, L1.2, U1.4 (FB)
- new net GND: C2.1, C3.1, C4.1, U1.1 (GND)
Other:
- title: ${BOARD_TITLE} -> Riddhi Buck 12V to 5V
